Commit message: Adapt joint limit of `Joint_2`
We operate solely in the *elbow up* configuration during control so that
users do not collide with table tops.

File: aria_description/urdf/aria_v2.urdf (robot description, URDF)
Before this commit: robot aria_v2_arm, 22 links, 21 joints
Joints:
- joint Joint_3: limit lower=-3.143 upper=1.689 effort=0 velocity=0.7 -> lower=-3.143 upper=-0.50 effort=0 velocity=0.7

Commit message: Adapt joint limit of `Joint_3`
That's a stable combination with the limits in `Joint_2` and avoids the
*diving*-like behavior when reaching the joint limits in Cartesian
control.

File: aria_description/urdf/aria_v2.urdf (robot description, URDF)
Before this commit: robot aria_v2_arm, 22 links, 21 joints
Joints:
- joint Joint_2: limit lower=-0.97 upper=3.615 effort=0 velocity=0.7 -> lower=0.33 upper=3.615 effort=0 velocity=0.7
